File: casing/fatherboard_oPMs.kicad_sch (KiCad schematic)
At the start: 16 parts, among them J0 - BATTERY, J1 + BATTERY, J2 SDA, J3 SCL, J4 GND, J5 3V3, J6 ULN_OUT, J7 ULN2003_VOUT, J8 VREG5.69V, J9 GPIOs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

Commit message: added LED signalling functionality started designing the web map, currently still WIP
Connections:
- net GP1: no longer U2.7 (I7)
Other:
- moved on the sheet: J2, J3, U2
